File: Hardware/SmartWatch/SmartWatch.sch (KiCad schematic (older format))
At the start: 47 parts, among them IC1 DA14683-00000U22, IC2 SPG08P4HM4H-1, IC3 MC3630, J1 Charging Port, M1 c0720b001f, Q1 ECH8693R-TL-W, Q2 ECH8693R-TL-W, U1 BQ297xy, U2 ATmega328P-MMH, U3 W25Q128JVS, U4 MAX30100EFD+, Y1 16Mhz, Y2 16Mhz, Y3 Crystal

Commit message: [Update] New footprints and new parts.
Change in the DA14683 footprint choice - bigger package will be used. Added programming connectors for DA14683 and ARDUINO R3. I2C and UART is being added.
Parts:
- removed IC1: DA14683-00000U22, BGA53C40P8X7_341X301X55, symbol SamacSys_Parts:DA14683-00000U22
- added AE1: Antenna, symbol Device:Antenna
- added C18: 100nF, Capacitor_SMD:C_01005_0402Metric, symbol Device:C
- added C19, C20: 10nF, Capacitor_SMD:C_01005_0402Metric, symbol Device:C
- added C21, C22: C, symbol Device:C
- added J2: Header_7, symbol Connector:Conn_01x07_Female
- added J3: ARD_PROG_CONN, symbol Connector:Conn_01x04_Female
- added JP1: Jumper, symbol Device:Jumper
- added L2: L, symbol Device:L
- added R13, R14, R15: 10K, Resistor_SMD:R_01005_0402Metric, symbol Device:R
- added R16, R17, R18: 3.3K, Resistor_SMD:R_01005_0402Metric, symbol Device:R
- added SW1: UP, symbol Switch:SW_MEC_5G
- added SW2: CHOOSE, symbol Switch:SW_MEC_5G
- added SW3: DOWN, symbol Switch:SW_MEC_5G
- added U5: DA14683-00000A92, XCVR_DA14680-01F08A92, symbol DA14683-00000A92:DA14683-00000A92
- C10, C11, C12, C13, C14, C15, C16, C17, C8, C9: footprint (none) -> Capacitor_SMD:C_01005_0402Metric
- C7: value C -> 100nF
- R11, R12: footprint (none) -> Resistor_SMD:R_01005_0402Metric
- Y2: footprint (none) -> Crystal:Crystal_SMD_HC49-SD
- Y3: value Crystal -> 32.768Mhz
Connections:
- net labels added: ARD_RST, ARD_RX, ARD_TX, LED2, LED3, P0_0, P0_1, P0_2, P0_3, P0_4, P0_5, P0_6, P0_7, P1_0, P1_1, P1_2, P1_3, P1_4, P1_5, P1_6, P2_0, P2_1, P2_2, P2_4, P3_0, P3_1, P3_2, P3_3, P3_4, P3_5, P3_6, P3_7, P4_0, P4_1, P4_2, P4_3, P4_4, P4_5, P4_6, P4_7, SCL, SDA, UART_RX, UART_TX
- net labels removed: ACCEL_SCL, ACCEL_SDA, ADC0_P1_2, ADC1_P1_4, ADC2_P1_3, ADC3_PO_7, ADC4_P0_6_PWM5, ADC5_P1_0, ADC6_P1_5, ADC7_P2_4, ARD_I2C_SCL, ARD_I2C_SDA, AVS1, AVS2, GND_BUCK, GND_RF1, GND_RF2, HEART_INT, HEART_SCL, HEART_SDA, MIC_CLK, MIC_DATA, MIC_SELECT, MOTOR_DRIVE, NTC_P1_6, PSUB_RF, QSPI_CLK, QSPI_CLK_P0_0, QSPI_CS_P0_5, QSPI_D0_P0_1, QSPI_D1_P0_2, QSPI_D2_P0_3, QSPI_D3_P0_4, QSPI_IO0, QSPI_IO1, QSPI_IO2, QSPI_IO3, SPEAKER_IN, USBN_P1_1, USBP_P2_2, VSS1, VSS2, VSS3, VSSIO1, VSSIO2, XTAL32KM_P2_1, XTAL32KP_P2_0
- wire segments 255 -> 301
Other:
- note added: "BUTTONS"
- moved on the sheet: C3, C4, C5, C6, IC2, L1, LS1, R11, R12, R8, U2, U3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

Commit message: [Update] Added CODEC and new Speaker and fixes
Parts:
- removed LS1: Speaker, symbol Device:Speaker
- added C? (x5): 0.1uF, symbol Device:C
- added C? (x5): 10uF, symbol Device:CP
- added IC1: 6PAIC3109TWRHMRQ1, QFN50P500X500X90-33N-D, symbol SamacSys_Parts:6PAIC3109TWRHMRQ1
- added LS1: SMS-1508MS-HT-R, SMS1508MSHTR, symbol SamacSys_Parts:SMS-1508MS-HT-R
Connections:
- wire segments 301 -> 332
Other:
- note added: "AUDIO CODEC"
- moved on the sheet: C18, C19, C20, C6, IC2, R13

Commit message: [Update] Added Display Connector
Added connector and fixed connector names.
Parts:
- added J?: Adafruit 4520, Connector_FFC-FPC:Hirose_FH12-24S-0.5SH_1x24-1MP_P0.50mm_Horizontal, symbol Connector:Conn_01x24_Female
- C21, C22, C? (x10): footprint (none) -> Capacitor_SMD:C_01005_0402Metric
- J2: value Header_7 -> DA_PROG_CONN
- JP1: footprint (none) -> Jumper:SolderJumper-2_P1.3mm_Bridged2Bar_Pad1.0x1.5mm
- L1: value 470nF -> 470nH; footprint (none) -> Inductor_SMD:L_0402_1005Metric
- L2: value L -> 470nH; footprint (none) -> Inductor_SMD:L_0402_1005Metric
Connections:
- net labels added: +3V3, CS, DB0, DB1, DB2, DB3, DB4, DB5, DB6, DB7, DC, IM12, IOVCC1.8V, LEDA, LEDK, NC, RD, RESET, SDIN, TE, VDD2.8V, WR
- wire segments 332 -> 364
Other:
- note added: "0"
- note added: "05/01/2022 (DD/MM/YYYY)"
- note removed: "01/10/2021 (DD/MM/YYYY)"
Changed lines of the file:
@@
 Smart Watch Schematic
 Text Notes 13000 11050 0    39   ~ 0
-01/10/2021 (DD/MM/YYYY)
+05/01/2022 (DD/MM/YYYY)
 Wire Wire Line
 	14250 1850 14250 1900
@@
 P 4300 2800
 F 0 "L1" H 4353 2846 50  0000 L CNN
-F 1 "470nF" H 4353 2755 50  0000 L CNN
-F 2 "" H 4300 2800 50  0001 C CNN
+F 1 "470nH" H 4353 2755 50  0000 L CNN
+F 2 "Inductor_SMD:L_0402_1005Metric" H 4300 2800 50  0001 C CNN
 F 3 "~" H 4300 2800 50  0001 C CNN
 	1    4300 2800
@@
 P 5700 2650
 F 0 "L2" V 5890 2650 50  0000 C CNN
-F 1 "L" V 5799 2650 50  0000 C CNN
-F 2 "" H 5700 2650 50  0001 C CNN
+F 1 "470nH" V 5799 2650 50  0000 C CNN
+F 2 "Inductor_SMD:L_0402_1005Metric" H 5700 2650 50  0001 C CNN
 F 3 "~" H 5700 2650 50  0001 C CNN
 	1    5700 2650
@@
 F 0 "C22" H 5900 2900 50  0000 L CNN
 F 1 "C" H 5900 2700 50  0000 L CNN
-F 2 "" H 5938 2650 50  0001 C CNN
+F 2 "Capacitor_SMD:C_01005_0402Metric" H 5938 2650 50  0001 C CNN
 F 3 "~" H 5900 2800 50  0001 C CNN
 	1    5900 2800
@@
 F 0 "C21" H 5550 2900 50  0000 L CNN
 F 1 "C" H 5550 2700 50  0000 L CNN
-F 2 "" H 5588 2650 50  0001 C CNN
+F 2 "Capacitor_SMD:C_01005_0402Metric" H 5588 2650 50  0001 C CNN
 F 3 "~" H 5550 2800 50  0001 C CNN
 	1    5550 2800
@@
 P 5350 3650
 F 0 "J2" H 5300 4050 50  0000 C CNN
-F 1 "Header_7" H 5150 4150 50  0000 C CNN
+F 1 "DA_PROG_CONN" H 5150 4150 50  0000 C CNN
 F 2 "" H 5350 3650 50  0001 C CNN
 F 3 "~" H 5350 3650 50  0001 C CNN
@@
 F 0 "JP1" V 14854 2727 50  0000 L CNN
 F 1 "Jumper" V 14945 2727 50  0000 L CNN
-F 2 "" H 14900 2600 50  0001 C CNN
+F 2 "Jumper:SolderJumper-2_P1.3mm_Bridged2Bar_Pad1.0x1.5mm" H 14900 2600 50  0001 C CNN
 F 3 "~" H 14900 2600 50  0001 C CNN
 	1    14900 2600
@@
 F 0 "C?" V 10600 5850 50  0000 C CNN
 F 1 "0.1uF" V 10650 6050 50  0000 C CNN
-F 2 "" H 10688 5600 50  0001 C CNN
+F 2 "Capacitor_SMD:C_01005_0402Metric" H 10688 5600 50  0001 C CNN
 F 3 "~" H 10650 5750 50  0001 C CNN
 	1    10650 5750
@@
 F 0 "C?" H 11400 7600 50  0000 C CNN
 F 1 "0.1uF" H 11350 7800 50  0000 C CNN
-F 2 "" H 11488 7550 50  0001 C CNN
+F 2 "Capacitor_SMD:C_01005_0402Metric" H 11488 7550 50  0001 C CNN
 F 3 "~" H 11450 7700 50  0001 C CNN
 	1    11450 7700
@@
 F 0 "C?" V 10600 5900 50  0000 C CNN
 F 1 "10uF" V 10600 5700 50  0000 C CNN
-F 2 "" H 10688 5850 50  0001 C CNN
+F 2 "Capacitor_SMD:C_01005_0402Metric" H 10688 5850 50  0001 C CNN
 F 3 "~" H 10650 6000 50  0001 C CNN
 	1    10650 6000
@@
 F 0 "C?" H 11250 7800 50  0000 C CNN
 F 1 "10uF" H 11300 7600 50  0000 C CNN
-F 2 "" H 11238 7550 50  0001 C CNN
+F 2 "Capacitor_SMD:C_01005_0402Metric" H 11238 7550 50  0001 C CNN
 F 3 "~" H 11200 7700 50  0001 C CNN
 	1    11200 7700
@@
 F 0 "C?" H 11400 7000 50  0000 C CNN
 F 1 "0.1uF" H 11350 7200 50  0000 C CNN
-F 2 "" H 11488 6950 50  0001 C CNN
+F 2 "Capacitor_SMD:C_01005_0402Metric" H 11488 6950 50  0001 C CNN
 F 3 "~" H 11450 7100 50  0001 C CNN
 	1    11450 7100
@@
 F 0 "C?" H 11250 7200 50  0000 C CNN
 F 1 "10uF" H 11300 7000 50  0000 C CNN
-F 2 "" H 11238 6950 50  0001 C CNN
+F 2 "Capacitor_SMD:C_01005_0402Metric" H 11238 6950 50  0001 C CNN
 F 3 "~" H 11200 7100 50  0001 C CNN
 	1    11200 7100
@@
 F 0 "C?" V 9350 6100 50  0000 C CNN
 F 1 "0.1uF" V 9400 6300 50  0000 C CNN
-F 2 "" H 9438 5850 50  0001 C CNN
+F 2 "Capacitor_SMD:C_01005_0402Metric" H 9438 5850 50  0001 C CNN
 F 3 "~" H 9400 6000 50  0001 C CNN
 	1    9400 6000
@@
 F 0 "C?" V 9350 5650 50  0000 C CNN
 F 1 "10uF" V 9350 5450 50  0000 C CNN
-F 2 "" H 9438 5600 50  0001 C CNN
+F 2 "Capacitor_SMD:C_01005_0402Metric" H 9438 5600 50  0001 C CNN
 F 3 "~" H 9400 5750 50  0001 C CNN
 	1    9400 5750
@@
 F 0 "C?" H 9250 7900 50  0000 C CNN
 F 1 "0.1uF" H 9200 8100 50  0000 C CNN
-F 2 "" H 9338 7850 50  0001 C CNN
+F 2 "Capacitor_SMD:C_01005_0402Metric" H 9338 7850 50  0001 C CNN
 F 3 "~" H 9300 8000 50  0001 C CNN
 	1    9300 8000
@@
 F 0 "C?" H 9100 8100 50  0000 C CNN
 F 1 "10uF" H 8950 7900 50  0000 C CNN
-F 2 "" H 9088 7850 50  0001 C CNN
+F 2 "Capacitor_SMD:C_01005_0402Metric" H 9088 7850 50  0001 C CNN
 F 3 "~" H 9050 8000 50  0001 C CNN
 	1    9050 8000
@@
 Text Notes 9400 5050 0    157  ~ 31
 AUDIO CODEC
+Text Notes 15450 11050 0    59   ~ 0
+0
+$Comp
+L Connector:Conn_01x24_Female J?
+U 1 1 61E28AE4
+P 9250 2650
+F 0 "J?" H 9142 1225 50  0000 C CNN
+F 1 "Adafruit 4520" H 9142 1316 50  0000 C CNN
+F 2 "Connector_FFC-FPC:Hirose_FH12-24S-0.5SH_1x24-1MP_P0.50mm_Horizontal" H 9250 2650 50  0001 C CNN
+F 3 "~" H 9250 2650 50  0001 C CNN
+	1    9250 2650
+	-1   0    0    1
+$EndComp
+Wire Wire Line
+	9450 1450 9800 1450
+Wire Wire Line
+	9450 1550 9800 1550
+Wire Wire Line
+	9450 1650 9800 1650
+Wire Wire Line
+	9450 1750 9800 1750
+Wire Wire Line
+	9450 1850 9800 1850
+Wire Wire Line
+	9450 1950 9800 1950
+Wire Wire Line
+	9450 2050 9800 2050
+Wire Wire Line
+	9450 2150 9800 2150
+Wire Wire Line
+	9450 2250 9800 2250
+Wire Wire Line
+	9450 2350 9800 2350
+Wire Wire Line
+	9450 2450 9800 2450
+Wire Wire Line
+	9450 2550 9800 2550
+Wire Wire Line
+	9450 2650 9800 2650
+Wire Wire Line
+	9450 2750 9800 2750
+Wire Wire Line
+	9450 2850 9800 2850
+Wire Wire Line
+	9450 2950 9800 2950
+Wire Wire Line
+	9450 3050 9800 3050
+Wire Wire Line
+	9450 3150 9800 3150
+Wire Wire Line
+	9450 3250 9800 3250
+Wire Wire Line
+	9450 3550 9800 3550
+Wire Wire Line
+	9450 3650 9800 3650
+Wire Wire Line
+	9450 3750 9800 3750
+Text Label 9450 3750 0    50   ~ 0
+LEDA
+Text Label 9450 3650 0    50   ~ 0
+LEDK
+Text Label 9450 3550 0    50   ~ 0
+GND
+Text Label 9450 3450 0    50   ~ 0
+VDD2.8V
+Text Label 9450 3350 0    50   ~ 0
+IOVCC1.8V
+Text Label 9450 3250 0    50   ~ 0
+IM12
+Text Label 9450 3150 0    50   ~ 0
+RESET
+Text Label 9450 3050 0    50   ~ 0
+CS
+Text Label 9450 2950 0    50   ~ 0
+DC
+Text Label 9450 2850 0    50   ~ 0
+WR
+Text Label 9450 2750 0    50   ~ 0
+RD
+Text Label 9450 2650 0    50   ~ 0
+SDIN
+Text Label 9450 2550 0    50   ~ 0
+DB0
+Text Label 9450 2450 0    50   ~ 0
+DB1
+Text Label 9450 2350 0    50   ~ 0
+DB2
+Text Label 9450 2250 0    50   ~ 0
+DB3
+Text Label 9450 2150 0    50   ~ 0
+DB4
+Text Label 9450 2050 0    50   ~ 0
+DB5
+Text Label 9450 1950 0    50   ~ 0
+DB6
+Text Label 9450 1850 0    50   ~ 0
+DB7
+Text Label 9450 1750 0    50   ~ 0
+TE
+Text Label 9450 1650 0    50   ~ 0
+NC
+Text Label 9450 1550 0    50   ~ 0
+GND
+Text Label 9450 1450 0    50   ~ 0
+GND
+Wire Wire Line
+	9800 1850 9800 1950
+Connection ~ 9800 1950
+Wire Wire Line
+	9800 1950 9800 2050
+Connection ~ 9800 2050
+Wire Wire Line
+	9800 2050 9800 2150
+Connection ~ 9800 2150
+Wire Wire Line
+	9800 2150 9800 2250
+Connection ~ 9800 2250
+Wire Wire Line
+	9800 2250 9800 2350
+Connection ~ 9800 2350
+Wire Wire Line
+	9800 2350 9800 2450
+Connection ~ 9800 2450
+Wire Wire Line
+	9800 2450 9800 2550
+$Comp
+L power:GND #PWR?
+U 1 1 61FD96DB
+P 9800 2150
+F 0 "#PWR?" H 9800 1900 50  0001 C CNN
+F 1 "GND" V 9800 1950 50  0000 C CNN
+F 2 "" H 9800 2150 50  0001 C CNN
+F 3 "" H 9800 2150 50  0001 C CNN
+	1    9800 2150
+	0    -1   -1   0
+$EndComp
+$Comp
+L power:GND #PWR?
+U 1 1 6200279B
+P 9800 3550
+F 0 "#PWR?" H 9800 3300 50  0001 C CNN
+F 1 "GND" V 9800 3350 50  0000 C CNN
+F 2 "" H 9800 3550 50  0001 C CNN
+F 3 "" H 9800 3550 50  0001 C CNN
+	1    9800 3550
+	0    -1   -1   0
+$EndComp
+$Comp
+L power:GND #PWR?
+U 1 1 6202B6ED
+P 9800 1450
+F 0 "#PWR?" H 9800 1200 50  0001 C CNN
+F 1 "GND" V 9800 1250 50  0000 C CNN
+F 2 "" H 9800 1450 50  0001 C CNN
+F 3 "" H 9800 1450 50  0001 C CNN
+	1    9800 1450
+	0    -1   -1   0
+$EndComp
+Wire Wire Line
+	9800 1450 9800 1550
+Connection ~ 9800 1450
+$Comp
+L power:+3V3 #PWR?
+U 1 1 6207F587
+P 9800 3450
+F 0 "#PWR?" H 9800 3300 50  0001 C CNN
+F 1 "+3V3" V 9815 3578 50  0000 L CNN
+F 2 "" H 9800 3450 50  0001 C CNN
+F 3 "" H 9800 3450 50  0001 C CNN
+	1    9800 3450
+	0    1    1    0
+$EndComp
+Wire Wire Line
+	9450 3350 9800 3350
+Wire Wire Line
+	9450 3450 9800 3450
+$Comp
+L power:+1V8 #PWR?
+U 1 1 6212A2FC
+P 9800 3350
+F 0 "#PWR?" H 9800 3200 50  0001 C CNN
+F 1 "+1V8" V 9815 3478 50  0000 L CNN
+F 2 "" H 9800 3350 50  0001 C CNN
+F 3 "" H 9800 3350 50  0001 C CNN
+	1    9800 3350
+	0    1    1    0
+$EndComp
 $EndSCHEMATC

Commit message: [Update] Full footprint assignment #1
Parts:
- AE1: footprint (none) -> RF_Antenna:Texas_SWRA117D_2.4GHz_Left
- J2: footprint (none) -> Connector_PinHeader_1.00mm:PinHeader_1x07_P1.00mm_Vertical_SMD_Pin1Left
- J3: footprint (none) -> Connector_PinHeader_1.00mm:PinHeader_1x04_P1.00mm_Vertical_SMD_Pin1Left
- SW1, SW2, SW3: footprint (none) -> Button_Switch_THT:SW_Tactile_SPST_Angled_PTS645Vx58-2LFS
- Y3: footprint (none) -> Crystal:Crystal_SMD_HC49-SD
Changed lines of the file:
@@
 F 0 "Y3" H 5750 2368 50  0000 C CNN
 F 1 "32.768Mhz" H 5750 2277 50  0000 C CNN
-F 2 "" H 5750 2100 50  0001 C CNN
+F 2 "Crystal:Crystal_SMD_HC49-SD" H 5750 2100 50  0001 C CNN
 F 3 "~" H 5750 2100 50  0001 C CNN
 	1    5750 2100
@@
 F 0 "AE1" H 5980 2439 50  0000 L CNN
 F 1 "Antenna" H 5980 2348 50  0000 L CNN
-F 2 "" H 5900 2450 50  0001 C CNN
+F 2 "RF_Antenna:Texas_SWRA117D_2.4GHz_Left" H 5900 2450 50  0001 C CNN
 F 3 "~" H 5900 2450 50  0001 C CNN
 	1    5900 2450
@@
 F 0 "J2" H 5300 4050 50  0000 C CNN
 F 1 "DA_PROG_CONN" H 5150 4150 50  0000 C CNN
-F 2 "" H 5350 3650 50  0001 C CNN
+F 2 "Connector_PinHeader_1.00mm:PinHeader_1x07_P1.00mm_Vertical_SMD_Pin1Left" H 5350 3650 50  0001 C CNN
 F 3 "~" H 5350 3650 50  0001 C CNN
 	1    5350 3650
@@
 F 0 "SW1" H 7000 10635 50  0000 C CNN
 F 1 "UP" H 7000 10544 50  0000 C CNN
-F 2 "" H 7000 10550 50  0001 C CNN
+F 2 "Button_Switch_THT:SW_Tactile_SPST_Angled_PTS645Vx58-2LFS" H 7000 10550 50  0001 C CNN
 F 3 "http://www.apem.com/int/index.php?controller=attachment&id_attachment=488" H 7000 10550 50  0001 C CNN
 	1    7000 10350
@@
 F 0 "SW2" H 7650 10635 50  0000 C CNN
 F 1 "CHOOSE" H 7650 10544 50  0000 C CNN
-F 2 "" H 7650 10550 50  0001 C CNN
+F 2 "Button_Switch_THT:SW_Tactile_SPST_Angled_PTS645Vx58-2LFS" H 7650 10550 50  0001 C CNN
 F 3 "http://www.apem.com/int/index.php?controller=attachment&id_attachment=488" H 7650 10550 50  0001 C CNN
 	1    7650 10350
@@
 F 0 "SW3" H 8300 10635 50  0000 C CNN
 F 1 "DOWN" H 8300 10544 50  0000 C CNN
-F 2 "" H 8300 10550 50  0001 C CNN
+F 2 "Button_Switch_THT:SW_Tactile_SPST_Angled_PTS645Vx58-2LFS" H 8300 10550 50  0001 C CNN
 F 3 "http://www.apem.com/int/index.php?controller=attachment&id_attachment=488" H 8300 10550 50  0001 C CNN
 	1    8300 10350
@@
 F 0 "J3" H 14642 3175 50  0000 C CNN
 F 1 "ARD_PROG_CONN" H 14642 3266 50  0000 C CNN
-F 2 "" H 14750 3600 50  0001 C CNN
+F 2 "Connector_PinHeader_1.00mm:PinHeader_1x04_P1.00mm_Vertical_SMD_Pin1Left" H 14750 3600 50  0001 C CNN
 F 3 "~" H 14750 3600 50  0001 C CNN
 	1    14750 3600

Commit message: [Update] Wired Display connector to MCU.
Communication type: SPI
Parts:
- removed SW1: UP, Button_Switch_THT:SW_Tactile_SPST_Angled_PTS645Vx58-2LFS, symbol Switch:SW_MEC_5G
- removed SW2: CHOOSE, Button_Switch_THT:SW_Tactile_SPST_Angled_PTS645Vx58-2LFS, symbol Switch:SW_MEC_5G
- removed SW3: DOWN, Button_Switch_THT:SW_Tactile_SPST_Angled_PTS645Vx58-2LFS, symbol Switch:SW_MEC_5G
- added SW1, SW2, SW3: SW_MEC_5E, Button_Switch_THT:SW_Tactile_SPST_Angled_PTS645Vx58-2LFS, symbol Switch:SW_MEC_5E
- BT1: footprint Battery:BatteryHolder_Keystone_3002_1x2032 -> Connector_PinHeader_1.00mm:PinHeader_1x02_P1.00mm_Vertical
- gave numbers to parts that had none: 11
Connections:
- wire segments 364 -> 368
- no-connect marks 11 -> 55
