File: Hardware/SmartWatch/SmartWatch.sch (KiCad schematic (older format))
At the start: 78 parts, among them IC1 6PAIC3109TWRHMRQ1, IC2 SPG08P4HM4H-1, IC3 MC3630, J1 Charging Port, J2 DA_PROG_CONN, J3 ARD_PROG_CONN, J4 Adafruit 4520, M1 c0720b001f, Q1 ECH8693R-TL-W, Q2 ECH8693R-TL-W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

Commit message: [Update] Fixed names of certain ICs.
Parts:
- U1: value BQ297xy -> BQ29700DSER
- U3: value W25Q128JVS -> W25Q128JVSIQ
- U4: value MAX30100EFD+ -> MAX30100EFD+T
Changed lines of the file:
@@
 P 2300 8600
 F 0 "U1" H 2300 8967 50  0000 C CNN
-F 1 "BQ297xy" H 2300 8876 50  0000 C CNN
+F 1 "BQ29700DSER" H 2300 8876 50  0000 C CNN
 F 2 "Package_SON:WSON-6_1.5x1.5mm_P0.5mm" H 2300 8950 50  0001 C CNN
 F 3 "http://www.ti.com/lit/ds/symlink/bq2970.pdf" H 2050 8800 50  0001 C CNN
@@
 P 7800 8200
 F 0 "U3" H 7800 8781 50  0000 C CNN
-F 1 "W25Q128JVS" H 7800 8690 50  0000 C CNN
+F 1 "W25Q128JVSIQ" H 7800 8690 50  0000 C CNN
 F 2 "Package_SO:SOIC-8_5.23x5.23mm_P1.27mm" H 7800 8200 50  0001 C CNN
 F 3 "http://www.winbond.com/resource-files/w25q128jv_dtr%20revc%2003272018%20plus.pdf" H 7800 8200 50  0001 C CNN
@@
 P 12800 5750
 F 0 "U4" H 13800 6137 60  0000 C CNN
-F 1 "MAX30100EFD+" H 13800 6031 60  0000 C CNN
+F 1 "MAX30100EFD+T" H 13800 6031 60  0000 C CNN
 F 2 "MAX30100:MAX30100EFD&plus_" H 13800 5990 60  0001 C CNN
 F 3 "" H 12800 5750 60  0000 C CNN

Commit message: [Update] Added BLE smartphone connection.
Parts:
- removed SW1: UP, Button_Switch_THT:SW_Tactile_SPST_Angled_PTS645Vx58-2LFS, symbol Switch:SW_MEC_5G
- removed SW2: CHOOSE, Button_Switch_THT:SW_Tactile_SPST_Angled_PTS645Vx58-2LFS, symbol Switch:SW_MEC_5G
- removed SW3: DOWN, Button_Switch_THT:SW_Tactile_SPST_Angled_PTS645Vx58-2LFS, symbol Switch:SW_MEC_5G
- added SW1: UP, Button_Switch_THT:SW_Tactile_SPST_Angled_PTS645Vx58-2LFS, symbol Switch:SW_Push
- added SW2: CHOOSE, Button_Switch_THT:SW_Tactile_SPST_Angled_PTS645Vx58-2LFS, symbol Switch:SW_Push
- added SW3: DOWN, Button_Switch_THT:SW_Tactile_SPST_Angled_PTS645Vx58-2LFS, symbol Switch:SW_Push
Changed lines of the file:
@@
 $EndComp
 Text Label 15000 3400 0    50   ~ 0
+ARD_TX
+Text Label 15000 3500 0    50   ~ 0
 ARD_RX
-Text Label 15000 3500 0    50   ~ 0
-ARD_TX
 Text Label 15000 3600 0    50   ~ 0
 ARD_RST
@@
 P3_2
 $Comp
-L Switch:SW_MEC_5G SW1
-U 1 1 61EEDF3D
-P 7000 10350
-F 0 "SW1" V 7046 10302 50  0000 R CNN
-F 1 "UP" V 6955 10302 50  0000 R CNN
-F 2 "Button_Switch_THT:SW_Tactile_SPST_Angled_PTS645Vx58-2LFS" H 7000 10550 50  0001 C CNN
-F 3 "http://www.apem.com/int/index.php?controller=attachment&id_attachment=488" H 7000 10550 50  0001 C CNN
-	1    7000 10350
-	0    -1   -1   0
-$EndComp
-$Comp
-L Switch:SW_MEC_5G SW2
-U 1 1 61F47DF6
-P 7650 10350
-F 0 "SW2" V 7696 10302 50  0000 R CNN
-F 1 "CHOOSE" V 7605 10302 50  0000 R CNN
-F 2 "Button_Switch_THT:SW_Tactile_SPST_Angled_PTS645Vx58-2LFS" H 7650 10550 50  0001 C CNN
-F 3 "http://www.apem.com/int/index.php?controller=attachment&id_attachment=488" H 7650 10550 50  0001 C CNN
-	1    7650 10350
-	0    -1   -1   0
-$EndComp
-$Comp
-L Switch:SW_MEC_5G SW3
-U 1 1 61F74894
-P 8300 10350
-F 0 "SW3" V 8346 10302 50  0000 R CNN
-F 1 "DOWN" V 8255 10302 50  0000 R CNN
-F 2 "Button_Switch_THT:SW_Tactile_SPST_Angled_PTS645Vx58-2LFS" H 8300 10550 50  0001 C CNN
-F 3 "http://www.apem.com/int/index.php?controller=attachment&id_attachment=488" H 8300 10550 50  0001 C CNN
-	1    8300 10350
-	0    -1   -1   0
-$EndComp
-$Comp
 L power:GNDREF #PWR0123
 U 1 1 61DDB960
@@
 Text Label 5350 2650 0    50   ~ 0
 RFIOP
+$Comp
+L Switch:SW_Push SW1
+U 1 1 6224D004
+P 7000 10350
+F 0 "SW1" V 7046 10302 50  0000 R CNN
+F 1 "UP" V 6955 10302 50  0000 R CNN
+F 2 "Button_Switch_THT:SW_Tactile_SPST_Angled_PTS645Vx58-2LFS" H 7000 10550 50  0001 C CNN
+F 3 "~" H 7000 10550 50  0001 C CNN
+	1    7000 10350
+	0    -1   -1   0
+$EndComp
+$Comp
+L Switch:SW_Push SW2
+U 1 1 622AB2C8
+P 7650 10350
+F 0 "SW2" V 7696 10302 50  0000 R CNN
+F 1 "CHOOSE" V 7605 10302 50  0000 R CNN
+F 2 "Button_Switch_THT:SW_Tactile_SPST_Angled_PTS645Vx58-2LFS" H 7650 10550 50  0001 C CNN
+F 3 "~" H 7650 10550 50  0001 C CNN
+	1    7650 10350
+	0    -1   -1   0
+$EndComp
+$Comp
+L Switch:SW_Push SW3
+U 1 1 622D7CC9
+P 8300 10350
+F 0 "SW3" V 8346 10302 50  0000 R CNN
+F 1 "DOWN" V 8255 10302 50  0000 R CNN
+F 2 "Button_Switch_THT:SW_Tactile_SPST_Angled_PTS645Vx58-2LFS" H 8300 10550 50  0001 C CNN
+F 3 "~" H 8300 10550 50  0001 C CNN
+	1    8300 10350
+	0    -1   -1   0
+$EndComp
 $EndSCHEMATC
