File: Hardware/SmartWatch/_autosave-SmartWatch.kicad_pcb (KiCad board)
At the start: 6 copper layers, 38.1 x 38.1 mm, 78 parts, among them IC1 6PAIC3109TWRHMRQ1, IC2 SPG08P4HM4H-1, IC3 MC3630, J1 Charging Port, J2 DA_PROG_CONN, J3 ARD_PROG_CONN, J4 Adafruit 4520, M1 c0720b001f, Q1 ECH8693R-TL-W, Q2 ECH8693R-TL-W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

Commit message: [Update] Changes to schematic and PCB test layout
Parts:
- moved L1 90.5 mm to (118.4, 77.5), turned to 90 degrees
Connections:
- L1 pad 2: /LA -> /LY
Routing:
- net /LX: track 0.00 -> 4.01 mm
Other:
- net class Default: clearance 0.2 -> 0.127; trace_width 0.25 -> 0.127
- rule trace_clearance: 0.2 -> 0.127
